File: Neopixel_Modules/Module_Large/Interactiles_Module_Neopixel.kicad_pcb (KiCad board)
At the start: 2 copper layers, 134.8 x 82.4 mm, 30 parts, among them J1 Screw_Terminal_2_P3.50mm, J2 PINHD_1x15_Male, J3 PINHD_1x15_Male, J4 PINHD_1x2_Female, SW1 SW_SPST

Commit message: fixed for pcb production
Connections:
- J3 pad GND: GND -> (no net)
- J3 pad MP: GND -> (no net)
Routing:
- net +5V: track 507.5 -> 564.4 mm, vias 0 -> 2
- net GND: track 0.00 -> 29.9 mm, vias 0 -> 8
- net SW11: track 174.8 -> 162.1 mm
Other:
- board text added: "1"
- board text added: "1 2 3 4 5 6 7 8 9 10 11 12 13 14 15"
- board text added: "10"
- board text added: "11"
- board text added: "12"
- board text added: "13"
- board text added: "14"
- board text added: "15"
- board text added: "2"
- board text added: "3"
- board text added: "4"
- board text added: "5"
- board text added: "6"
- board text added: "7"
- board text added: "8"
- board text added: "9"
- board text added: "LED OUT LED IN"
- board text removed: "< >"
